File: PCB/main/diva_main.kicad_pcb (KiCad board)
At the start: 2 copper layers, 273 x 97 mm, 59 parts, among them J1 Conn_01x04, K1 Conn_01x01_Female, K10 Conn_01x01_Female, K11 Conn_01x01_Female, K12 Conn_01x01_Female, K13 Conn_01x01_Female, K14 Conn_01x01_Female, K15 Conn_01x01_Female, K16 Conn_01x01_Female, K2 Conn_01x01_Female, K3 Conn_01x01_Female, K4 Conn_01x01_Female, K5 Conn_01x01_Female, K6 Conn_01x01_Female, K7 Conn_01x01_Female, K8 Conn_01x01_Female, K9 Conn_01x01_Female, U1 Pico_Trim, U3 MPR121QR2_BOARD, U4 MPR121QR2_BOARD, U8 SN74LV1T34DBV

Commit message: PCB layout done
Parts:
- removed U4: MPR121QR2_BOARD, diva_main:MPR121_BOARD
- added SW1: SWITCH_SPST, diva_main:SKSTAAE010, F.Cu at (341.5, 79.6)
- added SW2: SWITCH_SPST, diva_main:SKSTAAE010, F.Cu at (341.5, 89.6)
- added SW3: SWITCH_SPST, diva_main:SW_Kailh_Choc_V1V2_1.00u_LED, F.Cu at (300.5, 135.6)
- added SW4: SWITCH_SPST, diva_main:SW_Kailh_Choc_V1V2_1.00u_LED, F.Cu at (242.5, 135.6)
- added SW5: SWITCH_SPST, diva_main:SW_Kailh_Choc_V1V2_1.00u_LED, F.Cu at (184.5, 135.6)
- added SW6: SWITCH_SPST, diva_main:SW_Kailh_Choc_V1V2_1.00u_LED, F.Cu at (126.5, 135.6)
- added SW7: SWITCH_SPST, diva_main:B3F4000, F.Cu at (86.5, 84.6)
- added U2: MPR121QR2_BOARD, diva_main:MPR121_BOARD, B.Cu at (184.5, 106.6)
- moved D20 116.7 mm to (184.5, 130.9)
- moved D19 116.1 mm to (126.5, 146.6)
- moved D21 87.7 mm to (184.5, 146.6)
- moved D17 77.4 mm to (86.5, 74.6)
- moved D18 62.4 mm to (126.5, 130.9)
- moved U3 58.0 mm to (242.5, 106.6)
- moved D24 33.5 mm to (300.5, 130.9)
- moved D25 29.8 mm to (300.5, 146.6)
- moved D22 29.4 mm to (242.5, 130.9)
- moved D23 28.9 mm to (242.5, 146.6)
- moved R3 12.4 mm to (342.5, 71.6), turned to -90 degrees
- moved C5 11.6 mm to (115.5, 129.6), turned to 90 degrees
- moved U8 9.00 mm to (339.5, 71.6), turned to 90 degrees
- moved J1 8.06 mm to (95.5, 117.6), turned to 90 degrees
- moved C7 3.74 mm to (231.5, 129.6), turned to 90 degrees
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Connections:
- U3 pad 10: Net-(K3-Pin_1) -> Net-(K11-Pin_1)
- U3 pad 11: Net-(K4-Pin_1) -> Net-(K12-Pin_1)
- U3 pad 12: Net-(K5-Pin_1) -> Net-(K13-Pin_1)
- U3 pad 13: Net-(K6-Pin_1) -> Net-(K14-Pin_1)
- U3 pad 14: Net-(K7-Pin_1) -> Net-(K15-Pin_1)
- U3 pad 15: Net-(K8-Pin_1) -> Net-(K16-Pin_1)
- U3 pad 4: GND -> +3V3
- U3 pad 8: Net-(K1-Pin_1) -> Net-(K9-Pin_1)
- U3 pad 9: Net-(K2-Pin_1) -> Net-(K10-Pin_1)

Commit message: PCB v1.0 ready
Parts:
- moved D1 216.0 mm to (105.5, 57.6)
- moved D16 216.0 mm to (321.5, 57.6)
- moved D15 187.2 mm to (307.1, 57.6)
- moved D2 187.2 mm to (119.9, 57.6)
- moved D14 158.4 mm to (292.7, 57.6)
- moved D3 158.4 mm to (134.3, 57.6)
- moved D13 129.6 mm to (278.3, 57.6)
- moved D4 129.6 mm to (148.7, 57.6)
- moved D12 100.8 mm to (263.9, 57.6)
- moved D5 100.8 mm to (163.1, 57.6)
- moved D11 72.0 mm to (249.5, 57.6)
- moved D6 72.0 mm to (177.5, 57.6)
- moved U8 47.5 mm to (327.5, 117.6), turned to 180 degrees
- moved R3 45.5 mm to (327.5, 114.6), turned to 0 degrees
- moved D10 43.2 mm to (235.1, 57.6)
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- renumbered D24 to BL1, D25 to BL2, D22 to BL3, D23 to BL4, D20 to BL5, D21 to BL6, D18 to BL7, D19 to BL8, D17 to BL9
Connections:
- BL1 pad I: Net-(D23-Out) -> Net-(BL1-In)
- BL1 pad O: unconnected-(D24-Out-PadO) -> Net-(BL1-Out)
- BL2 pad I: Net-(D23-Out) -> Net-(BL1-In)
- BL3 pad I: Net-(D21-Out) -> Net-(BL1-Out)
- BL3 pad O: unconnected-(D22-Out-PadO) -> Net-(BL3-Out)
- BL4 pad I: Net-(D21-Out) -> Net-(BL1-Out)
- BL4 pad O: Net-(D23-Out) -> unconnected-(BL4-Out-PadO)
- BL5 pad I: Net-(D19-Out) -> Net-(BL3-Out)
- BL5 pad O: unconnected-(D20-Out-PadO) -> Net-(BL5-Out)
- BL6 pad I: Net-(D19-Out) -> Net-(BL3-Out)
- BL6 pad O: Net-(D21-Out) -> unconnected-(BL6-Out-PadO)
- BL7 pad I: Net-(D17-Out) -> Net-(BL5-Out)
- BL7 pad O: unconnected-(D18-Out-PadO) -> Net-(BL7-Out)
- BL8 pad I: Net-(D17-Out) -> Net-(BL5-Out)
- BL8 pad O: Net-(D19-Out) -> unconnected-(BL8-Out-PadO)
- BL9 pad I: Net-(D16-Out) -> Net-(BL7-Out)
- BL9 pad O: Net-(D17-Out) -> Net-(BL9-Out)
- C8 pad 1: +3V3 -> +5V
- D1 pad I: Net-(D1-In) -> Net-(BL9-Out)
- D16 pad O: Net-(D16-Out) -> unconnected-(D16-Out-PadO)
- R3 pad 1: Net-(D1-In) -> Net-(BL1-In)
- SW1 pad 1: unconnected-(SW1-"~{"}-Pad1) -> GND
- SW1 pad 2: unconnected-(SW1-"~{"}-Pad2) -> Net-(U1-GPIO1)
- SW2 pad 1: unconnected-(SW2-"~{"}-Pad1) -> GND
- SW2 pad 2: unconnected-(SW2-"~{"}-Pad2) -> Net-(U1-GPIO0)
- SW3 pad 1: unconnected-(SW3-"~{"}-Pad1) -> Net-(U1-GPIO9)
- SW3 pad 2: unconnected-(SW3-"~{"}-Pad2) -> GND
- SW4 pad 1: unconnected-(SW4-"~{"}-Pad1) -> Net-(U1-GPIO10)
- SW4 pad 2: unconnected-(SW4-"~{"}-Pad2) -> GND
- SW5 pad 1: unconnected-(SW5-"~{"}-Pad1) -> Net-(U1-GPIO11)
- SW5 pad 2: unconnected-(SW5-"~{"}-Pad2) -> GND
- SW6 pad 1: unconnected-(SW6-"~{"}-Pad1) -> Net-(U1-GPIO12)
- SW6 pad 2: unconnected-(SW6-"~{"}-Pad2) -> GND
- SW7 pad 1: unconnected-(SW7-"~{"}-Pad1) -> Net-(U1-GPIO13)
- SW7 pad 2: unconnected-(SW7-"~{"}-Pad2) -> GND
- U1 pad 1: unconnected-(U1-GPIO0-Pad1) -> Net-(U1-GPIO0)
- U1 pad 12: unconnected-(U1-GPIO9-Pad12) -> Net-(U1-GPIO9)
- U1 pad 14: unconnected-(U1-GPIO10-Pad14) -> Net-(U1-GPIO10)
- U1 pad 15: unconnected-(U1-GPIO11-Pad15) -> Net-(U1-GPIO11)
- U1 pad 16: unconnected-(U1-GPIO12-Pad16) -> Net-(U1-GPIO12)
- U1 pad 17: unconnected-(U1-GPIO13-Pad17) -> Net-(U1-GPIO13)
- U1 pad 2: unconnected-(U1-GPIO1-Pad2) -> Net-(U1-GPIO1)
- U8 pad 4: Net-(D1-In) -> Net-(BL1-In)
Routing:
- net +5V: track 0.00 -> 784.7 mm, vias 0 -> 12
- net +3V3: track 0.00 -> 289.8 mm, vias 0 -> 3
- net Net-(U1-GPIO13): track 0.00 -> 259.4 mm
- net /SDA: track 0.00 -> 224.9 mm, vias 0 -> 3
- net /SCL: track 0.00 -> 219.8 mm, vias 0 -> 3
- net Net-(U1-GPIO12): track 0.00 -> 206.7 mm
- net GND: track 0.00 -> 149.3 mm, vias 0 -> 29
- net Net-(U1-GPIO11): track 0.00 -> 147.7 mm
- net Net-(K16-Pin_1): track 0.00 -> 97.4 mm
- net Net-(U1-GPIO10): track 0.00 -> 88.7 mm
- net Net-(BL7-Out): track 0.00 -> 87.2 mm
- net Net-(K1-Pin_1): track 0.00 -> 86.5 mm
- net Net-(BL3-Out): track 0.00 -> 85.9 mm
- net Net-(BL1-Out): track 0.00 -> 85.7 mm
- net Net-(BL5-Out): track 0.00 -> 85.6 mm
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- added copper zone on B.Cu, net GND
- added copper zone on F.Cu, net GND
Other:
- board text added: "Diva Pico v1.0"
- board text added: "locked"

Commit message: PCB v1.1 (minor optimization)
Parts:
- removed R3: 10, Resistor_SMD:R_0603_1608Metric
- removed U8: SN74LV1T34DBV, diva_main:SOT-23-5_Jumper
Connections:
- U1 pad 4: Net-(U1-GPIO2) -> Net-(BL1-In)
Routing:
- net +5V: track 784.7 -> 762.6 mm
- net Net-(U1-GPIO2): track 18.3 -> 0.00 mm, vias 1 -> 0
- net Net-(BL1-In): track 54.5 -> 68.1 mm, vias 0 -> 1
- net GND: track 149.3 -> 145.4 mm
Other:
- board text added: "Diva Pico v1.1"
- board text added: "L"
- board text added: "R"
- board text added: "T O U C H S L I D E R"
- board text removed: "Diva Pico v1.0"
- board text removed: "locked"
