File: PCB/main/diva_main.kicad_sch (KiCad schematic)
At the start: 59 parts, among them J1 Conn_01x04, K1 Conn_01x01_Female, K10 Conn_01x01_Female, K11 Conn_01x01_Female, K12 Conn_01x01_Female, K13 Conn_01x01_Female, K14 Conn_01x01_Female, K15 Conn_01x01_Female, K16 Conn_01x01_Female, K2 Conn_01x01_Female, K3 Conn_01x01_Female, K4 Conn_01x01_Female, K5 Conn_01x01_Female, K6 Conn_01x01_Female, K7 Conn_01x01_Female, K8 Conn_01x01_Female, K9 Conn_01x01_Female, U1 Pico_Trim, U3 MPR121QR2_BOARD, U4 MPR121QR2_BOARD, U8 SN74LV1T34DBV

Commit message: PCB layout done
Parts:
- added SW1, SW2: SWITCH_SPST, diva_main:SKSTAAE010, symbol agg:SWITCH_SPST
- added SW3, SW4, SW5, SW6: SWITCH_SPST, diva_main:SW_Kailh_Choc_V1V2_1.00u_LED, symbol agg:SWITCH_SPST
- added SW7: SWITCH_SPST, diva_main:B3F4000, symbol agg:SWITCH_SPST
- renumbered U3 to U2, U4 to U3
Changed lines of the file:
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@@
+    )
+  )
+  (symbol (lib_id "agg:SWITCH_SPST") (at 111.76 113.03 90) (unit 1)
+    (in_bom yes) (on_board yes) (dnp no)
+    (property "Reference" "SW4" (at 112.395 113.03 90)
+      (effects (font (size 1.27 1.27)) (justify right))
+    )
+    (property "Value" "SWITCH_SPST" (at 113.03 114.2999 90)
+      (effects (font (size 1.27 1.27)) (justify right) hide)
+    )
+    (property "Footprint" "diva_main:SW_Kailh_Choc_V1V2_1.00u_LED" (at 111.76 113.03 0)
+      (effects (font (size 1.27 1.27)) hide)
+    )
+    (property "Datasheet" "" (at 111.76 113.03 0)
+      (effects (font (size 1.27 1.27)) hide)
+    )
+    (pin "1")
+    (pin "2")
+    (instances
+      (project "diva_main"
+        (path "/2e3f5573-c264-4a8b-a2f0-0e6473d39aad"
+          (reference "SW4") (unit 1)
+        )
+      )
     )
   )
@@
     )
   )
+  (symbol (lib_id "agg:SWITCH_SPST") (at 140.97 68.58 90) (unit 1)
+    (in_bom yes) (on_board yes) (dnp no)
+    (property "Reference" "SW2" (at 141.605 68.58 90)
+      (effects (font (size 1.27 1.27)) (justify right))
+    )
+    (property "Value" "SWITCH_SPST" (at 142.24 69.8499 90)
+      (effects (font (size 1.27 1.27)) (justify right) hide)
+    )
+    (property "Footprint" "diva_main:SKSTAAE010" (at 140.97 68.58 0)
+      (effects (font (size 1.27 1.27)) hide)
+    )
+    (property "Datasheet" "" (at 140.97 68.58 0)
+      (effects (font (size 1.27 1.27)) hide)
+    )
+    (pin "1")
+    (pin "2")
+    (instances
+      (project "diva_main"
+        (path "/2e3f5573-c264-4a8b-a2f0-0e6473d39aad"
+          (reference "SW2") (unit 1)
+        )
+      )
+    )
+  )
   (symbol (lib_id "Connector:Conn_01x01_Female") (at 311.15 120.65 0) (unit 1)
     (in_bom yes) (on_board yes) (dnp no)
@@
   (symbol (lib_id "diva_main:MPR121QR2_BOARD") (at 284.48 133.35 0) (unit 1)
     (in_bom yes) (on_board yes) (dnp no) (fields_autoplaced)
-    (property "Reference" "U4" (at 286.4994 110.49 0)
-      (effects (font (size 1.27 1.27)) (justify left))
-    )
-    (property "Value" "MPR121QR2_BOARD" (at 286.4994 113.03 0)
+    (property "Reference" "U3" (at 286.6741 110.49 0)
+      (effects (font (size 1.27 1.27)) (justify left))
+    )
+    (property "Value" "MPR121QR2_BOARD" (at 286.6741 113.03 0)
       (effects (font (size 1.27 1.27)) (justify left))
     )
@@
       (project "diva_main"
         (path "/2e3f5573-c264-4a8b-a2f0-0e6473d39aad"
-          (reference "U4") (unit 1)
+          (reference "U3") (unit 1)
         )
       )
@@
   (symbol (lib_id "diva_main:MPR121QR2_BOARD") (at 284.48 76.2 0) (unit 1)
     (in_bom yes) (on_board yes) (dnp no) (fields_autoplaced)
-    (property "Reference" "U3" (at 286.4994 53.34 0)
-      (effects (font (size 1.27 1.27)) (justify left))
-    )
-    (property "Value" "MPR121QR2_BOARD" (at 286.4994 55.88 0)
+    (property "Reference" "U2" (at 286.6741 53.34 0)
+      (effects (font (size 1.27 1.27)) (justify left))
+    )
+    (property "Value" "MPR121QR2_BOARD" (at 286.6741 55.88 0)
       (effects (font (size 1.27 1.27)) (justify left))
     )
@@
       (project "diva_main"
         (path "/2e3f5573-c264-4a8b-a2f0-0e6473d39aad"
-          (reference "U3") (unit 1)
+          (reference "U2") (unit 1)
         )
       )
@@
     )
   )
+  (symbol (lib_id "agg:SWITCH_SPST") (at 88.9 125.73 90) (unit 1)
+    (in_bom yes) (on_board yes) (dnp no)
+    (property "Reference" "SW6" (at 89.535 125.73 90)
+      (effects (font (size 1.27 1.27)) (justify right))
+    )
+    (property "Value" "SWITCH_SPST" (at 90.17 126.9999 90)
+      (effects (font (size 1.27 1.27)) (justify right) hide)
+    )
+    (property "Footprint" "diva_main:SW_Kailh_Choc_V1V2_1.00u_LED" (at 88.9 125.73 0)
+      (effects (font (size 1.27 1.27)) hide)
+    )
+    (property "Datasheet" "" (at 88.9 125.73 0)
+      (effects (font (size 1.27 1.27)) hide)
+    )
+    (pin "1")
+    (pin "2")
+    (instances
+      (project "diva_main"
+        (path "/2e3f5573-c264-4a8b-a2f0-0e6473d39aad"
+          (reference "SW6") (unit 1)
+        )
+      )
+    )
+  )
+  (symbol (lib_id "agg:SWITCH_SPST") (at 115.57 99.06 90) (unit 1)
+    (in_bom yes) (on_board yes) (dnp no)
+    (property "Reference" "SW3" (at 116.205 99.06 90)
+      (effects (font (size 1.27 1.27)) (justify right))
+    )
+    (property "Value" "SWITCH_SPST" (at 116.84 100.3299 90)
+      (effects (font (size 1.27 1.27)) (justify right) hide)
+    )
+    (property "Footprint" "diva_main:SW_Kailh_Choc_V1V2_1.00u_LED" (at 115.57 99.06 0)
+      (effects (font (size 1.27 1.27)) hide)
+    )
+    (property "Datasheet" "" (at 115.57 99.06 0)
+      (effects (font (size 1.27 1.27)) hide)
+    )
+    (pin "1")
+    (pin "2")
+    (instances
+      (project "diva_main"
+        (path "/2e3f5573-c264-4a8b-a2f0-0e6473d39aad"
+          (reference "SW3") (unit 1)
+        )
+      )
+    )
+  )
   (symbol (lib_id "power:GND") (at 179.07 219.71 0) (unit 1)
     (in_bom yes) (on_board yes) (dnp no)
@@
     )
   )
+  (symbol (lib_id "agg:SWITCH_SPST") (at 88.9 49.53 90) (unit 1)
+    (in_bom yes) (on_board yes) (dnp no)
+    (property "Reference" "SW7" (at 89.535 49.53 90)
+      (effects (font (size 1.27 1.27)) (justify right))
+    )
+    (property "Value" "SWITCH_SPST" (at 90.17 50.7999 90)
+      (effects (font (size 1.27 1.27)) (justify right) hide)
+    )
+    (property "Footprint" "diva_main:B3F4000" (at 88.9 49.53 0)
+      (effects (font (size 1.27 1.27)) hide)
+    )
+    (property "Datasheet" "" (at 88.9 49.53 0)
+      (effects (font (size 1.27 1.27)) hide)
+    )
+    (pin "1")
+    (pin "2")
+    (instances
+      (project "diva_main"
+        (path "/2e3f5573-c264-4a8b-a2f0-0e6473d39aad"
+          (reference "SW7") (unit 1)
+        )
+      )
+    )
+  )
   (symbol (lib_id "Connector:Conn_01x01_Female") (at 311.15 78.74 0) (unit 1)
     (in_bom yes) (on_board yes) (dnp no)
@@
         (path "/2e3f5573-c264-4a8b-a2f0-0e6473d39aad"
           (reference "K8") (unit 1)
+        )
+      )
+    )
+  )
+  (symbol (lib_id "agg:SWITCH_SPST") (at 106.68 124.46 90) (unit 1)
+    (in_bom yes) (on_board yes) (dnp no)
+    (property "Reference" "SW5" (at 107.315 124.46 90)
+      (effects (font (size 1.27 1.27)) (justify right))
+    )
+    (property "Value" "SWITCH_SPST" (at 107.95 125.7299 90)
+      (effects (font (size 1.27 1.27)) (justify right) hide)
+    )
+    (property "Footprint" "diva_main:SW_Kailh_Choc_V1V2_1.00u_LED" (at 106.68 124.46 0)
+      (effects (font (size 1.27 1.27)) hide)
+    )
+    (property "Datasheet" "" (at 106.68 124.46 0)
+      (effects (font (size 1.27 1.27)) hide)
+    )
+    (pin "1")
+    (pin "2")
+    (instances
+      (project "diva_main"
+        (path "/2e3f5573-c264-4a8b-a2f0-0e6473d39aad"
+          (reference "SW5") (unit 1)
         )
       )
@@
         )
       )
+    )
+  )
+  (symbol (lib_id "agg:SWITCH_SPST") (at 140.97 59.69 90) (unit 1)
+    (in_bom yes) (on_board yes) (dnp no)
+    (property "Reference" "SW1" (at 141.605 59.69 90)
+      (effects (font (size 1.27 1.27)) (justify right))
+    )
+    (property "Value" "SWITCH_SPST" (at 142.24 60.9599 90)
+      (effects (font (size 1.27 1.27)) (justify right) hide)
+    )
+    (property "Footprint" "diva_main:SKSTAAE010" (at 140.97 59.69 0)
+      (effects (font (size 1.27 1.27)) hide)
+    )
+    (property "Datasheet" "" (at 140.97 59.69 0)
+      (effects (font (size 1.27 1.27)) hide)
+    )
+    (pin "1")
+    (pin "2")
+    (instances
+      (project "diva_main"
+        (path "/2e3f5573-c264-4a8b-a2f0-0e6473d39aad"
+          (reference "SW1") (unit 1)
+        )
+      )

Commit message: PCB v1.0 ready
Parts:
- renumbered D17 to BL1, D18 to BL2, D19 to BL3, D20 to BL4, D21 to BL5, D22 to BL6, D23 to BL7, D24 to BL8, D25 to BL9
Connections:
- net +3V3: no longer C8.1
- net +5V: now also C8.1
- net GND: now also SW1.1 ("~{"}), SW2.1 ("~{"}), SW3.2 ("~{"}), SW4.2 ("~{"}), SW5.2 ("~{"}), SW6.2 ("~{"}), SW7.2 ("~{"})
- net at SW4.1 ("~{"}): now also U1.14 (GPIO10)
- net at BL7.O (Out), BL9.I (In): no longer BL8.I (In)
- net at BL3.O (Out), BL5.I (In): now also BL6.I (In); no longer BL4.I (In)
- net at BL5.O (Out), BL7.I (In): now also BL8.I (In); no longer BL6.I (In)
- net at R3.1, U8.4 (Y): now also BL1.I (In), BL2.I (In); no longer D1.I (In)
- net at U1.1 (GPIO0): now also SW2.2 ("~{"})
- net at U1.12 (GPIO9): now also SW3.1 ("~{"})
- net at U1.15 (GPIO11): now also SW5.1 ("~{"})
- net at U1.16 (GPIO12): now also SW6.1 ("~{"})
- net at U1.17 (GPIO13): now also SW7.1 ("~{"})
- net at U1.2 (GPIO1): now also SW1.2 ("~{"})
- net at BL9.O (Out): now also D1.I (In)
- net at BL1.O (Out), BL3.I (In): now also BL4.I (In); no longer BL2.I (In)
- net at D16.O (Out): no longer BL1.I (In)
- no-connect marks 39 -> 36
Other:
- moved on the sheet: BL1, BL2, BL3, BL4, BL5, BL6, BL7, BL8, BL9, C1, C2, C3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

Commit message: PCB v1.1 (minor optimization)
Parts:
- removed R3: 10, Resistor_SMD:R_0603_1608Metric, symbol Device:R_Small
- removed U8: SN74LV1T34DBV, diva_main:SOT-23-5_Jumper, symbol Logic_LevelTranslator:SN74LV1T34DBV
Connections:
- net at BL1.I (In), BL2.I (In): now also U1.4 (GPIO2)
