File: PCB/plus/diva_plus.kicad_sch (KiCad schematic)
At the start: 114 parts, among them K1 Conn_01x01_Female, K10 Conn_01x01_Female, K11 Conn_01x01_Female, K12 Conn_01x01_Female, K13 Conn_01x01_Female, K14 Conn_01x01_Female, K15 Conn_01x01_Female, K16 Conn_01x01_Female, K17 Conn_01x01_Female, K18 Conn_01x01_Female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

Commit message: Diva Pico+ files
Connections:
- net +5V is gone; now on net VLED: C1.1, C2.1, C3.1, C4.1, C5.1, C6.1, C7.1, C8.1, D1.V (VDD), D10.V (VDD), D11.V (VDD), D12.V (VDD)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
