File: PCB/plus/diva_plus.kicad_pcb (KiCad board)
At the start: 2 copper layers, 357.8 x 137.8 mm, 114 parts, among them K1 Conn_01x01_Female, K10 Conn_01x01_Female, K11 Conn_01x01_Female, K12 Conn_01x01_Female, K13 Conn_01x01_Female, K14 Conn_01x01_Female, K15 Conn_01x01_Female, K16 Conn_01x01_Female, K17 Conn_01x01_Female, K18 Conn_01x01_Female, K19 Conn_01x01_Female, K2 Conn_01x01_Female, K20 Conn_01x01_Female, K21 Conn_01x01_Female, K22 Conn_01x01_Female, K23 Conn_01x01_Female, K24 Conn_01x01_Female, K25 Conn_01x01_Female, K26 Conn_01x01_Female, K27 Conn_01x01_Female, K28 Conn_01x01_Female, K29 Conn_01x01_Female, K3 Conn_01x01_Female, K30 Conn_01x01_Female, K31 Conn_01x01_Female, K32 Conn_01x01_Female, K4 Conn_01x01_Female, K5 Conn_01x01_Female, K6 Conn_01x01_Female, K7 Conn_01x01_Female, K8 Conn_01x01_Female, K9 Conn_01x01_Female, SW1 SWITCH_SPST, SW2 SWITCH_SPST, SW3 SWITCH_SPST, SW4 SWITCH_SPST, SW5 SWITCH_SPST, SW6 SWITCH_SPST, SW7 SWITCH_SPST, U1 Pico_Trim, U2 MPR121QR2_BOARD, U3 MPR121QR2_BOARD, U4 MPR121QR2_BOARD, U5 LM4040DBZ-2.1, U6 LP5907MFX-4.2, U7 ADG704BRUZ

Commit message: Diva Pico+ files
Parts:
- C1, C12, C2, C3, C4, C5, C6, C7, C8: moved to B.Cu
- moved C12 48.6 mm to (81.2, 189.7)
- moved R1 32.1 mm to (335.0, 143.6)
- moved R2 32.1 mm to (335.0, 141.6)
- moved Z1 32.1 mm to (334.5, 139.1)
- moved C11 30.3 mm to (327.7, 138.6)
- moved U7 30.3 mm to (324.7, 141.6)
- moved U2 30.0 mm to (139.0, 125.6)
- moved U4 30.0 mm to (295.0, 125.6)
- moved C5 22.5 mm to (346.1, 161.6)
- moved C6 22.5 mm to (268.1, 161.6)
- moved C7 22.5 mm to (190.1, 161.6)
- moved C8 22.5 mm to (112.1, 161.6)
- moved U3 10.0 mm to (217.0, 125.6)
- moved U5 4.12 mm to (386.0, 115.6), turned to 0 degrees
- moved U1 0.80 mm to (368.8, 131.6)
Connections:
- C1 pad 1: +5V -> VLED
- C2 pad 1: +5V -> VLED
- C3 pad 1: +5V -> VLED
- C4 pad 1: +5V -> VLED
- C5 pad 1: +5V -> VLED
- C6 pad 1: +5V -> VLED
- C7 pad 1: +5V -> VLED
- C8 pad 1: +5V -> VLED
- D1 pad V: +5V -> VLED
- D10 pad V: +5V -> VLED
- D11 pad V: +5V -> VLED
- D12 pad V: +5V -> VLED
- D13 pad V: +5V -> VLED
- D14 pad V: +5V -> VLED
- D15 pad V: +5V -> VLED
- D16 pad V: +5V -> VLED
- D17 pad V: +5V -> VLED
- D18 pad V: +5V -> VLED
- D19 pad V: +5V -> VLED
- D2 pad V: +5V -> VLED
- D20 pad V: +5V -> VLED
- D21 pad V: +5V -> VLED
- D22 pad V: +5V -> VLED
- D23 pad V: +5V -> VLED
- D24 pad V: +5V -> VLED
- D25 pad V: +5V -> VLED
- D26 pad V: +5V -> VLED
- D27 pad V: +5V -> VLED
- D28 pad V: +5V -> VLED
- D29 pad V: +5V -> VLED
- D3 pad V: +5V -> VLED
- D30 pad V: +5V -> VLED
- D31 pad V: +5V -> VLED
- D32 pad V: +5V -> VLED
- D4 pad V: +5V -> VLED
- D5 pad V: +5V -> VLED
- D6 pad V: +5V -> VLED
- D7 pad V: +5V -> VLED
- D8 pad V: +5V -> VLED
- D9 pad V: +5V -> VLED
Routing:
- net VLED: track 297.7 -> 1590.7 mm, vias 16 -> 21
- net VHall: track 3.88 -> 553.5 mm, vias 0 -> 9
- net +5V: track 472.1 -> 0.00 mm, vias 2 -> 0
- net +3V3: track 0.00 -> 276.6 mm, vias 0 -> 5
- net /S4: track 0.00 -> 250.4 mm, vias 0 -> 2
- net /S3: track 0.00 -> 160.7 mm, vias 0 -> 2
- net GND: track 66.9 -> 206.3 mm, vias 8 -> 129
- net /S2: track 0.00 -> 90.5 mm, vias 0 -> 2
- net Net-(BL11-Out): track 77.6 -> 136.3 mm
- net Net-(U1-GPIO26_ADC0): track 83.6 -> 49.9 mm, vias 0 -> 2
- net Net-(K11-Pin_1): track 65.2 -> 33.8 mm
- net /S1: track 0.00 -> 30.5 mm
- net Net-(K1-Pin_1): track 55.0 -> 85.0 mm
- net Net-(U1-GPIO18): track 73.8 -> 43.9 mm, vias 0 -> 2
- net Net-(K31-Pin_1): track 52.6 -> 82.5 mm
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- added copper zone on B.Cu, net GND
- added copper zone on F.Cu, net GND
Other:
- outline, holes or cut-outs redrawn

Commit message: Minor footprint and silkscreen finetune
Other:
- board text added: "Diva Pico+ v1.01"
- board text removed: "Diva Pico+ v1.0"
Changed lines of the file:
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@@
 		)
 		(fp_rect
-			(start -1.8 1.5)
-			(end 1.8 -1.5)
+			(start -1.75 1.45)
+			(end 1.75 -1.45)
 			(stroke
 				(width 0.15)
@@
 		)
 		(fp_rect
-			(start -1.8 1.5)
-			(end 1.8 -1.5)
+			(start -1.75 1.45)
+			(end 1.75 -1.45)
 			(stroke
 				(width 0.15)
@@
 		)
 		(fp_rect
-			(start -1.8 1.5)
-			(end 1.8 -1.5)
+			(start -1.75 1.45)
+			(end 1.75 -1.45)
 			(stroke
 				(width 0.15)
@@
 		)
 		(fp_rect
-			(start -1.8 1.5)
-			(end 1.8 -1.5)
+			(start -1.75 1.45)
+			(end 1.75 -1.45)
 			(stroke
 				(width 0.15)
@@
 		)
 		(fp_rect
-			(start -1.8 1.5)
-			(end 1.8 -1.5)
+			(start -1.75 1.45)
+			(end 1.75 -1.45)
 			(stroke
 				(width 0.15)
@@
 		)
 		(fp_rect
-			(start -1.8 1.5)
-			(end 1.8 -1.5)
+			(start -1.75 1.45)
+			(end 1.75 -1.45)
 			(stroke
 				(width 0.15)
@@
 		)
 		(fp_rect
-			(start -1.8 1.5)
-			(end 1.8 -1.5)
+			(start -1.75 1.45)
+			(end 1.75 -1.45)
 			(stroke
 				(width 0.15)
@@
 		)
 		(fp_rect
-			(start -1.8 1.5)
-			(end 1.8 -1.5)
+			(start -1.75 1.45)
+			(end 1.75 -1.45)
 			(stroke
 				(width 0.15)
@@
 		)
 		(fp_rect
-			(start -1.8 1.5)
-			(end 1.8 -1.5)
+			(start -1.75 1.45)
+			(end 1.75 -1.45)
 			(stroke
 				(width 0.15)
@@
 		)
 		(fp_rect
-			(start -1.8 1.5)
-			(end 1.8 -1.5)
+			(start -1.75 1.45)
+			(end 1.75 -1.45)
 			(stroke
 				(width 0.15)
@@
 		)
 		(fp_rect
-			(start -1.8 1.5)
-			(end 1.8 -1.5)
+			(start -1.75 1.45)
+			(end 1.75 -1.45)
 			(stroke
 				(width 0.15)
@@
 		)
 		(fp_rect
-			(start -1.8 1.5)
-			(end 1.8 -1.5)
+			(start -1.75 1.45)
+			(end 1.75 -1.45)
 			(stroke
 				(width 0.15)
@@
 		)
 		(fp_rect
-			(start -1.8 1.5)
-			(end 1.8 -1.5)
+			(start -1.75 1.45)
+			(end 1.75 -1.45)
 			(stroke
 				(width 0.15)
@@
 		)
 		(fp_rect
-			(start -1.8 1.5)
-			(end 1.8 -1.5)
+			(start -1.75 1.45)
+			(end 1.75 -1.45)
 			(stroke
 				(width 0.15)
@@
 		)
 		(fp_rect
-			(start -1.8 1.5)
-			(end 1.8 -1.5)
+			(start -1.75 1.45)
+			(end 1.75 -1.45)
 			(stroke
 				(width 0.15)
@@
 		)
 		(fp_rect
-			(start -1.8 1.5)
-			(end 1.8 -1.5)
+			(start -1.75 1.45)
+			(end 1.75 -1.45)
 			(stroke
 				(width 0.15)
@@
 		)
 		(fp_rect
-			(start -1.8 1.5)
-			(end 1.8 -1.5)
+			(start -1.75 1.45)
+			(end 1.75 -1.45)
 			(stroke
 				(width 0.15)
@@
 	)
 	(gr_text "github.com/whowechina"
-		(at 47.966 135.71268 0)
+		(at 48.356 137.37268 0)
 		(layer "F.SilkS")
 		(effects
@@
 	(gr_text "L"
 		(locked yes)
-		(at 78.986685 100.39268 0)
+		(at 79.236 100.39268 0)
 		(layer "F.SilkS" knockout)
 		(effects
@@
 			(polygon
 				(pts
-					(xy 87.398897 98.94768) (xy 82.142302 98.94768) (xy 81.548404 98.894132) (xy 81.12266 98.752553)
-					(xy 80.822444 98.539733) (xy 80.608999 98.240091) (xy 80.467107 97.815341) (xy 80.41346 97.222989)
-					(xy 80.41346 91.279217) (xy 80.463587 90.951827) (xy 80.608091 90.68702) (xy 80.753351 90.554288)
-					(xy 80.935953 90.47307) (xy 81.16759 90.444121) (xy 81.406947 90.473329) (xy 81.592997 90.554676)
-					(xy 81.738508 90.686501) (xy 81.88303 90.951239) (xy 81.933139 91.278179) (xy 81.933139 97.000331)
-					(xy 81.970719 97.271772) (xy 82.064969 97.426962) (xy 82.22344 97.517111) (xy 82.487448 97.552564)
-					(xy 87.398897 97.552564) (xy 87.694251 97.597982) (xy 87.938673 97.730068) (xy 88.061745 97.863131)
-					(xy 88.137363 98.032641) (xy 88.164445 98.250122) (xy 88.137363 98.467603) (xy 88.061745 98.637113)
-					(xy 87.938673 98.770176) (xy 87.694251 98.902261)
+					(xy 87.648212 98.94768) (xy 82.391617 98.94768) (xy 81.797719 98.894132) (xy 81.371975 98.752553)
+					(xy 81.071759 98.539733) (xy 80.858314 98.240091) (xy 80.716422 97.815341) (xy 80.662775 97.222989)
+					(xy 80.662775 91.279217) (xy 80.712902 90.951827) (xy 80.857406 90.68702) (xy 81.002666 90.554288)
+					(xy 81.185268 90.47307) (xy 81.416905 90.444121) (xy 81.656262 90.473329) (xy 81.842312 90.554676)
+					(xy 81.987823 90.686501) (xy 82.132345 90.951239) (xy 82.182454 91.278179) (xy 82.182454 97.000331)
+					(xy 82.220034 97.271772) (xy 82.314284 97.426962) (xy 82.472755 97.517111) (xy 82.736763 97.552564)
+					(xy 87.648212 97.552564) (xy 87.943566 97.597982) (xy 88.187988 97.730068) (xy 88.31106 97.863131)
+					(xy 88.386678 98.032641) (xy 88.41376 98.250122) (xy 88.386678 98.467603) (xy 88.31106 98.637113)
+					(xy 88.187988 98.770176) (xy 87.943566 98.902261)
 				)
 			)
 		)
 	)
-	(gr_text "Diva Pico+ v1.0"
-		(at 47.436 132.34268 0)
+	(gr_text "Diva Pico+ v1.01"
+		(at 44.936 134.23268 0)
 		(layer "F.SilkS")
 		(effects
@@
 	)
 	(zone
+		(net 70)
+		(net_name "Net-(U1-GPIO9)")
+		(layer "F.Cu")
+		(name "$teardrop_padvia$")
+		(hatch none 0.1)
+		(priority 30000)
+		(attr
+			(teardrop
+				(type padvia)
+			)
+		)
+		(connect_pads yes
+			(clearance 0)
+		)
+		(min_thickness 0.0254)
+		(filled_areas_thickness no)
+		(fill yes
+			(thermal_gap 0.5)
+			(thermal_bridge_width 0.5)
+			(island_removal_mode 1)
+			(island_area_min 10)
+		)
+		(polygon
+			(pts
+				(xy 336.114864 167.69268) (xy 336.114864 167.29268) (xy 334.647127 166.578063) (xy 334.035 167.49268)
+				(xy 334.647127 168.407297)
+			)
+		)
+	)
+	(zone
 		(net 73)
 		(net_name "Net-(U1-GPIO12)")
@@
 	)
 	(zone
-		(net 70)
-		(net_name "Net-(U1-GPIO9)")
+		(net 72)
+		(net_name "Net-(U1-GPIO11)")
 		(layer "F.Cu")
 		(name "$teardrop_padvia$")
 		(hatch none 0.1)
-		(priority 30000)
+		(priority 30002)
 		(attr
 			(teardrop
@@
 		(polygon
 			(pts
-				(xy 336.114864 167.69268) (xy 336.114864 167.29268) (xy 334.647127 166.578063) (xy 334.035 167.49268)
-				(xy 334.647127 168.407297)
+				(xy 180.114864 167.69268) (xy 180.114864 167.29268) (xy 178.647127 166.578063) (xy 178.035 167.49268)
+				(xy 178.647127 168.407297)
 			)
 		)
 	)
 	(zone
-		(net 72)
-		(net_name "Net-(U1-GPIO11)")
+		(net 71)
+		(net_name "Net-(U1-GPIO10)")
 		(layer "F.Cu")
 		(name "$teardrop_padvia$")
 		(hatch none 0.1)
-		(priority 30002)
+		(priority 30001)
 		(attr
 			(teardrop
@@
 		(polygon
 			(pts
-				(xy 180.114864 167.69268) (xy 180.114864 167.29268) (xy 178.647127 166.578063) (xy 178.035 167.49268)
-				(xy 178.647127 168.407297)
+				(xy 258.114864 167.69268) (xy 258.114864 167.29268) (xy 256.647127 166.578063) (xy 256.035 167.49268)
+				(xy 256.647127 168.407297)
 			)
 		)
@@
 			)
 		)
-	)
-	(zone
-		(net 71)
-		(net_name "Net-(U1-GPIO10)")
-		(layer "F.Cu")
-		(name "$teardrop_padvia$")
-		(hatch none 0.1)
-		(priority 30001)
-		(attr
-			(teardrop
-				(type padvia)
-			)
-		)
-		(connect_pads yes
-			(clearance 0)
-		)
-		(min_thickness 0.0254)
-		(filled_areas_thickness no)
-		(fill yes
-			(thermal_gap 0.5)
-			(thermal_bridge_width 0.5)
-			(island_removal_mode 1)
-			(island_area_min 10)
-		)
-		(polygon
-			(pts
-				(xy 258.114864 167.69268) (xy 258.114864 167.29268) (xy 256.647127 166.578063) (xy 256.035 167.49268)
-				(xy 256.647127 168.407297)
-			)
-		)
